Commit message: 하드코딩 포기. vla 넣어보자.

File: open_manipulator/open_manipulator_description/urdf/omy_f3m/omy_f3m.urdf (robot description, URDF)
Before this commit: robot omy_f3m, 17 links, 16 joints
Links:
- removed link camera_bottom_screw_frame
- added link camera_color_optical_frame
Joints:
- removed joint camera_joint
- removed joint camera_link_joint
- added joint camera_fixed: type fixed, parent end_effector_flange_link, child camera_link, origin xyz=0.013 0.00 0.07 rpy=0 0 0
- added joint camera_optical_fixed: type fixed, parent camera_link, child camera_color_optical_frame, origin xyz=0 0 0 rpy=-1.57079632679 0 -1.57079632679

File: open_manipulator/open_manipulator_description/urdf/omy_f3m/omy_f3m_arm.urdf.xacro (robot description, xacro)
@@ -2,5 +2,4 @@
 <robot xmlns:xacro="http://www.ros.org/wiki/xacro">
    <xacro:macro name="omy_f3m" params="prefix">
-      <xacro:include filename="$(find realsense2_description)/urdf/_d405.urdf.xacro" />
       <xacro:property name="meshes_file_direction" value="package://open_manipulator_description/meshes/omy_f3m" />
       <link name="${prefix}link0">
@@ -206,6 +205,7 @@
          </inertial>
       </link>
-      <xacro:sensor_d405 parent="${prefix}link6" use_nominal_extrinsics="false" name="${prefix}camera">
-         <origin xyz="-0.021 -0.07385 0.0803" rpy="-1.57079632679 0 -1.57079632679"/>
+      <xacro:include filename="$(find realsense2_description)/urdf/_d405.urdf.xacro" />
+      <xacro:sensor_d405 parent="${prefix}end_effector_flange_link" use_nominal_extrinsics="false" name="${prefix}camera">
+         <origin xyz="0.013 0.00 0.07" rpy="0 0 0"/>
       </xacro:sensor_d405>
       <joint name="${prefix}end_effector_flange_joint" type="fixed">
